Commit message: Actualizado subs de cmd y envia comuniacion a arduino

File: src/install/diffbot_description/share/diffbot_description/urdf/diffbot.urdf.xacro (robot description, xacro)
@@ -29,5 +29,5 @@
         <mesh filename="package://diffbot_description/meshes/Chasis.stl" />
       </geometry>
-      <material name="blue"/>
+      <material name="white"/>
     </visual>
     <inertial>
@@ -102,10 +102,10 @@
         </inertial>
       </link>
-    <joint name="${prefix}caster_frontal_wheel_joint" type="fixed">
+    <!--joint name="${prefix}caster_frontal_wheel_joint" type="fixed">
       <parent link="${prefix}base_link"/>
       <child link="${prefix}caster_frontal_wheel"/>
       <origin xyz="${base_width/2 - caster_wheel_radius} 0 ${z_offset}" rpy="0 0 0"/>
     </joint>
-    <!-- caster frontal wheel Link -->
+    < caster frontal wheel Link >
     <link name="${prefix}caster_frontal_wheel">
       <collision>
@@ -130,5 +130,5 @@
           izz="${caster_wheel_mass * 0.4 * (caster_wheel_radius * caster_wheel_radius)}"/>
         </inertial>
-      </link>
+      </link-->
     <joint name="${prefix}caster_rear_wheel_joint" type="fixed">
       <parent link="${prefix}base_link"/>

Commit message: Ya se puede ver el Rover en Gazebo
Falta terminar de ponerlo bien y hacer el launch, también se tuvo que instalar algunas librerias para probar el LIDAR

File: src/install/diffbot_description/share/diffbot_description/urdf/diffbot.urdf.xacro (robot description, xacro)
@@ -43,5 +43,6 @@
       <parent link="${prefix}base_link"/>
       <child link="${prefix}left_wheel"/>
-      <origin xyz="0.126 -${(base_width/2) + 0.036} 0.18" rpy="0 0 0"/>
+      <!--origin xyz="0.126 -${(base_width/2) + 0.036} 0.18" rpy="0 0 0"/-->
+      <origin xyz="-0.19 -${base_width/2} -${base_height}" rpy="0 0 0"/>
       <axis xyz="0 1 0"/>
       <dynamics damping="0.2"/>
@@ -58,5 +59,6 @@
         <origin xyz="0 0 0" rpy="${PI/2} 0 0"/>
         <geometry>
-          <cylinder length="${wheel_len}" radius="${wheel_radius}"/>
+          <!--cylinder length="${wheel_len}" radius="${wheel_radius}"/-->
+          <mesh filename="package://diffbot_description/meshes/Orugas.stl" />
         </geometry>
         <material name="black"/>
@@ -74,5 +76,6 @@
       <parent link="${prefix}base_link"/>
       <child link="${prefix}right_wheel"/>
-      <origin xyz="0.126 ${(base_width/2) +0.036} 0.18" rpy="0 0 0"/>
+      <!--origin xyz="0.126 ${(base_width/2) +0.06} 0.18" rpy="0 0 0"/-->
+      <origin xyz="-0.19 ${base_width/2+0.10} -${base_height}" rpy="0 0 0"/>
       <axis xyz="0 1 0"/>
       <dynamics damping="0.2"/>
@@ -89,5 +92,6 @@
         <origin xyz="0 0 0" rpy="${PI/2} 0 0"/>
         <geometry>
-          <cylinder length="${wheel_len}" radius="${wheel_radius}"/>
+          <!--cylinder length="${wheel_len}" radius="${wheel_radius}"/-->
+          <mesh filename="package://diffbot_description/meshes/Orugas.stl" />
         </geometry>
         <material name="black"/>
